Commit message: Comple Tssk 1 setup Nav2 for simulation and real robots(starbots cleaner 2) and testing #1-241004

File: rb1_ros2/rb1_ros2_description/urdf/elevator/elevator.gazebo.xacro (robot description, xacro)
@@ -8,20 +8,16 @@
 			<kd value="1.0" />
 			<fdir1 value="1 0 0"/>
-			<material>Gazebo/Black</material>
+			<!-- <material>Gazebo/Black</material> -->
+			<material>Gazebo/Yellow</material>
 			<turnGravityOff>false</turnGravityOff>
-			<!--kp>500000.0</kp>
-			<kd>10.0</kd>
+			<!-- <kp>5000000.0</kp>
+			<kd>10000.0</kd>
 			<mu1>10</mu1>
 			<mu2>10</mu2>
-			<fdir1>1 0 0</fdir1-->
-			<!--minDepth>0.001</minDepth-->
-			<!--material>Gazebo/Black</material-->
-			<!--mu1 value="10"/>
-			<mu2 value="5"/>
-			<kp value="500000.0" />
-			<kd value="10.0" />
-			<fdir1 value="1 0 0"/>
-			<material>Gazebo/Yellow</material>
-			<turnGravityOff>false</turnGravityOff-->
+			<fdir1>1 0 0</fdir1>
+			<minDepth>0.005</minDepth> -->
+			<!-- <material>Gazebo/Black</material> -->
+			<!-- <material>Gazebo/Yellow</material>
+			<turnGravityOff>false</turnGravityOff> -->
 		</gazebo>
 		<!--gazebo reference="${name}_wheel_link">

File: rb1_ros2/rb1_ros2_description/urdf/wheels/rubber_wheel.gazebo.xacro (robot description, xacro)
@@ -2,5 +2,5 @@
 <robot xmlns:xacro="http://www.ros.org/wiki/xacro">
 	<xacro:macro name="rubber_wheel_gazebo" params="prefix">
-		<!-- <gazebo reference="${prefix}wheel_link">
+		<gazebo reference="${prefix}wheel_link">
 			<mu1 value="5.0"/>
 			<mu2 value="0.5"/>
@@ -9,5 +9,5 @@
 			<fdir1 value="1 0 0"/>
     		<material>Gazebo/Yellow</material>
-			<turnGravityOff>false</turnGravityOff> -->
+			<turnGravityOff>false</turnGravityOff>
 			<!--kp>500000.0</kp>
 			<kd>10.0</kd>
@@ -24,6 +24,6 @@
 			<material>Gazebo/Yellow</material>
 			<turnGravityOff>false</turnGravityOff-->
-		<!-- </gazebo> -->
-		<gazebo reference="${prefix}wheel_link">
+		</gazebo>
+		<!-- <gazebo reference="${prefix}wheel_link">
 			<kp>1000.0</kp>
 			<kd>100000.0</kd>
@@ -35,6 +35,6 @@
 			<material>Gazebo/Yellow</material>
 			<turnGravityOff>true</turnGravityOff>
-			<!-- <implicitSpringDamper>1</implicitSpringDamper> -->
-		</gazebo>
+			<implicitSpringDamper>1</implicitSpringDamper>
+		</gazebo> -->
 	</xacro:macro>
 </robot>

File: rb1_ros2/rb1_ros2_description/urdf/wheels/rubber_wheel.urdf.xacro (robot description, xacro)
@@ -50,5 +50,5 @@
         </geometry>
 <!-- for increasing rolling friction -->
-		<surface>
+		<!-- <surface>
 			<bounce>
 				<restitution_coefficient>.5</restitution_coefficient>
@@ -70,4 +70,5 @@
 			</contact>
 		</surface>
+ -->
       </collision>
       <inertial>

File: rb1_ros2/rb1_ros2_description/xacro/rb1_ros2_base.urdf.xacro (robot description, xacro)
@@ -27,14 +27,18 @@
 	<xacro:property name="wheel_offset_y" value="0.218" />
 	<!-- <xacro:property name="wheel_offset_z" value="0.0512" /> -->
-	<xacro:property name="wheel_offset_z" value="0.050" />
+	<!-- <xacro:property name="wheel_offset_z" value="0.050" /> -->
+	<xacro:property name="wheel_offset_z" value="0.0512" />
 	<!-- Castor paramters -->
 	<xacro:property name="omni_back_x" value="0.195" />
 	<xacro:property name="omni_back_y" value="0.0" />
+	<xacro:property name="omni_back_z" value="0.0260" />
 	<!-- <xacro:property name="omni_back_z" value="0.0270" /> -->
-	<xacro:property name="omni_back_z" value="0.032" />
+	<!-- <xacro:property name="omni_back_z" value="0.032" /> -->
+	<!-- <xacro:property name="omni_back_z" value="0.031" /> -->
 	<xacro:property name="omni_front_x" value="0.132" />
 	<xacro:property name="omni_front_y" value="0.1535" />
 	<!-- <xacro:property name="omni_front_z" value="0.0270" /> -->
-	<xacro:property name="omni_front_z" value="0.032" />
+	<!-- <xacro:property name="omni_front_z" value="0.032" /> -->
+	<xacro:property name="omni_front_z" value="0.031" />
     <!-- ******************* -->
 	<!-- ELEVATOR PARAMETERS -->
