Commit message: Working on Task2-3-4 in sim and testing#1

File: rb1_ros2/rb1_ros2_description/xacro/rb1_ros2_base.urdf.xacro (robot description, xacro)
@@ -26,12 +26,11 @@
 	<!-- x,y,z in translation from base_link to the center of the wheel -->
 	<xacro:property name="wheel_offset_y" value="0.218" />
-	<!-- <xacro:property name="wheel_offset_z" value="0.0512" /> -->
-	<!-- <xacro:property name="wheel_offset_z" value="0.050" /> -->
-	<xacro:property name="wheel_offset_z" value="0.0512" />
+    <!-- <xacro:property name="wheel_offset_z" value="0.0512" /> -->
+    <xacro:property name="wheel_offset_z" value="0.054" />
 	<!-- Castor paramters -->
 	<xacro:property name="omni_back_x" value="0.195" />
 	<xacro:property name="omni_back_y" value="0.0" />
+	<!-- <xacro:property name="omni_back_z" value="0.0270" /> -->
 	<xacro:property name="omni_back_z" value="0.0260" />
-	<!-- <xacro:property name="omni_back_z" value="0.0270" /> -->
 	<!-- <xacro:property name="omni_back_z" value="0.032" /> -->
 	<!-- <xacro:property name="omni_back_z" value="0.031" /> -->
@@ -39,6 +38,6 @@
 	<xacro:property name="omni_front_y" value="0.1535" />
 	<!-- <xacro:property name="omni_front_z" value="0.0270" /> -->
-	<!-- <xacro:property name="omni_front_z" value="0.032" /> -->
-	<xacro:property name="omni_front_z" value="0.031" />
+	<!-- <xacro:property name="omni_front_z" value="0.031" /> -->
+	<xacro:property name="omni_front_z" value="0.034" />
     <!-- ******************* -->
 	<!-- ELEVATOR PARAMETERS -->

Commit message: Complet Task 2,3,4 and wep app in simulation env robots and testing #2-241105

File: rb1_ros2/rb1_ros2_description/xacro/rb1_ros2_base.urdf.xacro (robot description, xacro)
@@ -39,5 +39,6 @@
 	<!-- <xacro:property name="omni_front_z" value="0.0270" /> -->
 	<!-- <xacro:property name="omni_front_z" value="0.031" /> -->
-	<xacro:property name="omni_front_z" value="0.034" />
+	<!-- <xacro:property name="omni_front_z" value="0.034" /> -->
+	<xacro:property name="omni_front_z" value="0.035" />
     <!-- ******************* -->
 	<!-- ELEVATOR PARAMETERS -->
