Commit message: Complete Task 5-docker and testing #4-241202

File: rb1_ros2/rb1_ros2_description/urdf/common.gazebo.xacro (robot description, xacro)
@@ -7,7 +7,4 @@
                 <robot_param_node>/rb1_robot/robot_state_publisher</robot_param_node>
                 <parameters>$(find rb1_ros2_description)/config/rb1_controller.yaml</parameters>
-                <ros>
-                    <remapping>/controller_manager/robot_description:=/rb1_robot/robot_description</remapping>
-                </ros>
             </plugin>
         </gazebo>

File: rb1_ros2/rb1_ros2_description/urdf/elevator/elevator.gazebo.xacro (robot description, xacro)
@@ -8,29 +8,7 @@
 			<kd value="1.0" />
 			<fdir1 value="1 0 0"/>
-			<!-- <material>Gazebo/Black</material> -->
 			<material>Gazebo/Yellow</material>
 			<turnGravityOff>false</turnGravityOff>
-			<!-- <kp>5000000.0</kp>
-			<kd>10000.0</kd>
-			<mu1>10</mu1>
-			<mu2>10</mu2>
-			<fdir1>1 0 0</fdir1>
-			<minDepth>0.005</minDepth> -->
-			<!-- <material>Gazebo/Black</material> -->
-			<!-- <material>Gazebo/Yellow</material>
-			<turnGravityOff>false</turnGravityOff> -->
 		</gazebo>
-		<!--gazebo reference="${name}_wheel_link">
-			<kp>500000.0</kp>
-			<kd>10.0</kd>
-			<mu1>10</mu1>
-			<mu2>10</mu2>
-			<fdir1>1 0 0</fdir1>
-			<maxVel>1.0</maxVel>
-			<minDepth>0.003</minDepth>
-			<material>Gazebo/Yellow</material>
-			<turnGravityOff>false</turnGravityOff>
-			<implicitSpringDamper>1</implicitSpringDamper>
-		</gazebo-->
 	</xacro:macro>
 </robot>

File: rb1_ros2/rb1_ros2_description/urdf/elevator/elevator.urdf.xacro (robot description, xacro)
@@ -9,13 +9,4 @@
     </xacro:macro>
 	<xacro:macro name="elevator_platform" params="prefix parent hq *origin">
-	<!-- PARAMS: -->
-	<!-- name : name of the link: -->
-	<!-- hq: selects model in high quality (.dae) -->
-    <!-- <xacro:macro name="solid_cuboid_inertia1" params="m h d w">
-		<inertia  ixx="${(m*(h*h+d*d))/12}" ixy = "0" ixz = "0"
-              iyy="${(m*(w*w+d*d))/12}" iyz = "0"
-              izz="${(m*(w*w+h*h))/12}"
-        />
-    </xacro:macro> -->
 	<!-- ELEVATOR_BASE_LINK -->
 	<!-- <joint name="${prefix}_base_joint" type="fixed"> -->
@@ -26,11 +17,4 @@
 	</joint>
 	<link name="${prefix}_base_link">
-		<!--inertial>
-			<mass value="0.1" />
-			<origin xyz="0 0 0" />
-			<inertia	ixx="0.007" ixy="0.0"  ixz="0.0"
-						iyy="0.007"  iyz="0.0"
-						izz="0.78125"/>
-		</inertial-->
 		<inertial>
 			<mass value="2" />
@@ -72,9 +56,4 @@
 	</joint>
 	<link name="${prefix}_platform_link">
-		<!--inertial>
-			<mass value="0.05" />
-			<origin xyz="0 0 0" />
-			<inertia  ixx="0.00007" ixy="0.0"  ixz="0.0"  iyy="0.00007"  iyz="0.0"  izz="0.0078" />
-		</inertial-->
 		<inertial>
 			<mass value="2" />

File: rb1_ros2/rb1_ros2_description/urdf/hokuyo_ust20lx.urdf.xacro (robot description, xacro)
@@ -26,11 +26,4 @@
       </inertial>
     </link>
-    <!-- <link name="${prefix}_link">
-	  </link>
-    <joint name="${prefix}_joint" type="fixed">
-      <parent link="${prefix}_base_link"/>
-      <child link="${prefix}_link"/>
-      <origin xyz="0.00 0.0 0.0474" rpy="0 0 0"/>
-	  </joint> -->
     <!-- Hokuyo sensor for simulation -->
     <xacro:sensor_hokuyo_ust20_gazebo/>
@@ -62,7 +55,5 @@
                     <min>0.06</min>
                     <max>20.0</max>
-                    <!-- resolution>0.004363323</resolution -->
                     <resolution>0.004359297</resolution>
-                    <!-- resolution>0.001</resolution -->
                 </range>
                 <noise>

File: rb1_ros2/rb1_ros2_description/urdf/wheels/omni_wheel.urdf.xacro (robot description, xacro)
@@ -46,10 +46,4 @@
         </geometry>
       </collision>
-      <!--collision>
-      <origin xyz="0 0 0" rpy="${M_PI/2} 0 0" />
-       <geometry>
-         <sphere radius="${omni_wheel_radius}"/>
-       </geometry>
-     </collision-->
       <inertial>
         <mass value="${wheel_mass}" />
@@ -68,16 +62,4 @@
 		<turnGravityOff>false</turnGravityOff>
     </gazebo>
-    <!--gazebo reference="${name}_wheel">
-		<kp>500000.0</kp>
-		<kd>10.0</kd>
-		<mu1>10</mu1>
-		<mu2>10</mu2>
-		<fdir1>1 0 0</fdir1>
-		<maxVel>1.0</maxVel>
-		<minDepth>0.003</minDepth>
-		<material>Gazebo/Black</material>
-		<turnGravityOff>false</turnGravityOff>
-		<implicitSpringDamper>1</implicitSpringDamper>
-    </gazebo-->
   </xacro:macro>
 </robot>

File: rb1_ros2/rb1_ros2_description/urdf/wheels/rubber_wheel.gazebo.xacro (robot description, xacro)
@@ -10,31 +10,5 @@
     		<material>Gazebo/Yellow</material>
 			<turnGravityOff>false</turnGravityOff>
-			<!--kp>500000.0</kp>
-			<kd>10.0</kd>
-			<mu1>10</mu1>
-			<mu2>10</mu2>
-			<fdir1>1 0 0</fdir1-->
-			<!--minDepth>0.001</minDepth-->
-			<!--material>Gazebo/Black</material-->
-			<!--mu1 value="10"/>
-			<mu2 value="5"/>
-			<kp value="500000.0" />
-			<kd value="10.0" />
-			<fdir1 value="1 0 0"/>
-			<material>Gazebo/Yellow</material>
-			<turnGravityOff>false</turnGravityOff-->
 		</gazebo>
-		<!-- <gazebo reference="${prefix}wheel_link">
-			<kp>1000.0</kp>
-			<kd>100000.0</kd>
-			<mu1>100</mu1>
-			<mu2>100</mu2>
-			<fdir1>1 0 0</fdir1>
-			<maxVel>1.0</maxVel>
-			<minDepth>0.005</minDepth>
-			<material>Gazebo/Yellow</material>
-			<turnGravityOff>true</turnGravityOff>
-			<implicitSpringDamper>1</implicitSpringDamper>
-		</gazebo> -->
 	</xacro:macro>
 </robot>

File: rb1_ros2/rb1_ros2_description/urdf/wheels/rubber_wheel.urdf.xacro (robot description, xacro)
@@ -49,26 +49,4 @@
           <cylinder length="${wheel_height}" radius="${wheel_radius}" />
         </geometry>
-<!-- for increasing rolling friction -->
-		<!-- <surface>
-			<bounce>
-				<restitution_coefficient>.5</restitution_coefficient>
-			</bounce>
-			<friction>
-				<ode>
-					<mu>10</mu>
-					<mu2>10</mu2>
-					<fdir1>1 0 0</fdir1>
-					<slip1>0</slip1>
-					<slip2>0</slip2>
-				</ode>
-			</friction>
-			<contact>
-				<ode>
-                    <kp>1e15</kp>
-                    <kd>1e13</kd>
-                </ode>
-			</contact>
-		</surface>
- -->
       </collision>
       <inertial>

File: rb1_ros2/rb1_ros2_description/xacro/rb1_ros2_base.urdf.xacro (robot description, xacro)
@@ -87,10 +87,4 @@
 		<origin xyz="0.210 0.0 0.21" rpy="0 3.1416 3.1416"/>
 	</xacro:sensor_hokuyo_ust20lx>
-	<!-- <xacro:sensor_imu_hector prefix="$(arg prefix)imu" parent="$(arg prefix)base_link">
-		<origin xyz="0.002 0.053 0.1485" rpy="0 0 0"/>
-	</xacro:sensor_imu_hector> -->
-	<!-- <xacro:sensor_orbbec_astra prefix="$(arg prefix)front_rgbd_camera" parent="$(arg prefix)base_link" prefix_topic="front_rgbd_camera">
-		<origin xyz="0.234 0.0 0.092" rpy="0 0 0"/>
-	</xacro:sensor_orbbec_astra> -->
     <gazebo reference="$(arg prefix)front_laser_base_link">
         <sensor name="lidar" type="ray">
@@ -120,5 +114,4 @@
           <plugin name="scan" filename="libgazebo_ros_ray_sensor.so">
               <ros>
-                  <!-- <namespace>${robot_name}</namespace> -->
                   <remapping>~/out:=scan</remapping>
               </ros>
@@ -131,6 +124,6 @@
     <xacro:ros2_control_gazebo/>
     <!-- ROS2 control - diff drive -->
-    <ros2_control name="diff_drive" type="system">
-        <hardware>
+    <ros2_control name="diff_drive_test" type="system">
+        <hardware name="diff_drive_test">
           <plugin>gazebo_ros2_control/GazeboSystem</plugin>
         </hardware>
@@ -156,5 +149,5 @@
     <!-- ROS2 control - position -->
     <ros2_control name="joint_position" type="system">
-        <hardware>
+        <hardware name="joint_position">
             <plugin>gazebo_ros2_control/GazeboSystem</plugin>
         </hardware>
